File: hardware/launch_clock_pcb_v3_demo/launch_clock_pcb_v3_demo.kicad_pcb (KiCad board)
At the start: 4 copper layers, 126.1 x 43.6 mm, 48 parts, among them J1 lc_USB-C_2, U1 ATmega328P, U2 MAX7221, U3 MAX7221, U4 DS3231M, U5 CP2102N-Axx-xQFN24, U6 AP22816BKWT, U7 USBLC6-2SC6, X1 16MHz

Commit message: Fix custom KiCad library paths
Parts:
- J1: value lc_USB-C_2 -> SAMESKY_UJ20-C-H-G-SMT-1-P16-TR
- S2: value lc_reset_button -> SW_TS18-5-25-SL-260-SMT-TR
